File: PortablePower/PortablePower.kicad_pcb (KiCad board)
At the start: 2 copper layers, 9.3 x 6 mm, 7 parts, among them IC1 SW6208, J1 USB1130-15-A, J2 2137160001

Commit message: before done schematic
Parts:
- added C10: 22uf, Capacitor_SMD:C_1210_3225Metric_Pad1.33x2.70mm_HandSolder, F.Cu at (110.0, 80.5)
- added C11: 22uf/10v, Capacitor_SMD:C_0603_1608Metric_Pad1.08x0.95mm_HandSolder, F.Cu at (121.1, 58.3)
- added C12: 0.1uf, Capacitor_SMD:C_0805_2012Metric_Pad1.18x1.45mm_HandSolder, F.Cu at (142.0, 84.4)
- added C4: 10uf, Capacitor_SMD:C_1210_3225Metric_Pad1.33x2.70mm_HandSolder, F.Cu at (110.0, 59.2)
- added C5: 10uf, Capacitor_SMD:C_1210_3225Metric_Pad1.33x2.70mm_HandSolder, F.Cu at (110.0, 63.5)
- added C6: 22uf, Capacitor_SMD:C_1210_3225Metric_Pad1.33x2.70mm_HandSolder, F.Cu at (110.0, 67.7)
- added C7: 0.1uf, Capacitor_SMD:C_0805_2012Metric_Pad1.18x1.45mm_HandSolder, F.Cu at (125.3, 68.6)
- added C8: 22uf, Capacitor_SMD:C_1210_3225Metric_Pad1.33x2.70mm_HandSolder, F.Cu at (110.0, 72.0)
- added C9: 22uf, Capacitor_SMD:C_1210_3225Metric_Pad1.33x2.70mm_HandSolder, F.Cu at (110.0, 76.2)
- added D1: LED, LED_SMD:LED_1206_3216Metric_Pad1.42x1.75mm_HandSolder, F.Cu at (116.0, 58.8)
- added D2: LED, LED_SMD:LED_1206_3216Metric_Pad1.42x1.75mm_HandSolder, F.Cu at (116.0, 62.2)
- added D3: LED, LED_SMD:LED_1206_3216Metric_Pad1.42x1.75mm_HandSolder, F.Cu at (116.0, 65.6)
- added D4: LED, LED_SMD:LED_1206_3216Metric_Pad1.42x1.75mm_HandSolder, F.Cu at (116.0, 68.9)
- added D5: LED, LED_SMD:LED_1206_3216Metric_Pad1.42x1.75mm_HandSolder, F.Cu at (116.0, 72.3)
- added D6: LED, LED_SMD:LED_1206_3216Metric_Pad1.42x1.75mm_HandSolder, F.Cu at (116.0, 75.7)
- added Q1: CSD17313Q2, Package_SON:Texas_DQK, F.Cu at (120.9, 69.0)
- added Q2: CSD17313Q2, Package_SON:Texas_DQK, F.Cu at (120.9, 72.7)
- added Q3: CSD16406Q3, CSD16406Q3:DQG_VSON-CLIP, F.Cu at (123.4, 100.8)
- added Q4: CSD16406Q3, CSD16406Q3:DQG_VSON-CLIP, F.Cu at (127.9, 100.8)
- added R1: 5m ohm, Resistor_SMD:R_1206_3216Metric_Pad1.30x1.75mm_HandSolder, F.Cu at (121.9, 80.2)
- added R2: 10k, Resistor_SMD:R_0603_1608Metric_Pad0.98x0.95mm_HandSolder, F.Cu at (121.1, 60.8)
- added R3: 10k, Resistor_SMD:R_0603_1608Metric_Pad0.98x0.95mm_HandSolder, F.Cu at (121.1, 63.4)
- added R4: 330, Resistor_SMD:R_0805_2012Metric_Pad1.20x1.40mm_HandSolder, F.Cu at (125.3, 71.6)
- added R5: 26.7k, Resistor_SMD:R_0603_1608Metric_Pad0.98x0.95mm_HandSolder, F.Cu at (121.1, 65.9)
- added R6: 330, Resistor_SMD:R_0805_2012Metric_Pad1.20x1.40mm_HandSolder, F.Cu at (123.5, 111.5)
- added R7: 2.2k, Resistor_SMD:R_0603_1608Metric_Pad0.98x0.95mm_HandSolder, F.Cu at (124.2, 95.0)
- added R8: 5M, Resistor_SMD:R_1206_3216Metric_Pad1.30x1.75mm_HandSolder, F.Cu at (124.1, 105.0)
- added R9: 5M, Resistor_SMD:R_1206_3216Metric_Pad1.30x1.75mm_HandSolder, F.Cu at (124.1, 108.3)
- added S1: B3U1000P, B3U1000P:B3U-1000P, F.Cu at (115.6, 79.3)
- added TP1: NTC, Connector_PinHeader_2.00mm:PinHeader_2x01_P2.00mm_Vertical, F.Cu at (121.0, 76.5)
- added TP10: DATA, TestPoint:TestPoint_Pad_D1.0mm, F.Cu at (90.2, 104.4)
- added TP11: CCL/WLED, TestPoint:TestPoint_Pad_D1.0mm, F.Cu at (90.2, 107.5)
- added TP12: B-, TestPoint:TestPoint_Pad_D4.0mm, F.Cu at (118.1, 101.6)
- added TP13: B+, TestPoint:TestPoint_Pad_4.0x4.0mm, F.Cu at (118.1, 107.6)
- added TP2: VBUSL, TestPoint:TestPoint_Pad_D1.0mm, F.Cu at (87.2, 95.3)
- added TP3: VBUSS2, TestPoint:TestPoint_Pad_D1.0mm, F.Cu at (87.2, 98.3)
- added TP4: VOUTA2, TestPoint:TestPoint_Pad_D1.0mm, F.Cu at (87.2, 101.4)
- added TP5: DMA2, TestPoint:TestPoint_Pad_D1.0mm, F.Cu at (87.2, 104.4)
- added TP6: DPA2, TestPoint:TestPoint_Pad_D1.0mm, F.Cu at (87.2, 107.5)
- added TP7: DPB, TestPoint:TestPoint_Pad_D1.0mm, F.Cu at (90.2, 95.3)
- added TP8: DMB, TestPoint:TestPoint_Pad_D1.0mm, F.Cu at (90.2, 98.3)
- added TP9: VBUSB, TestPoint:TestPoint_Pad_D1.0mm, F.Cu at (90.2, 101.4)
- added U1: USBLC6-2SC6, Package_TO_SOT_SMD:SOT-23-6, F.Cu at (125.9, 59.5)
- added U2: USBLC6-2SC6, Package_TO_SOT_SMD:SOT-23-6, F.Cu at (125.9, 64.1)
- added U3: BQ297xy, Package_SON:WSON-6_1.5x1.5mm_P0.5mm, F.Cu at (127.6, 111.7)
Connections:
- C1 pad 1: +VDC -> +BATT
- C2 pad 1: +VDC -> +BATT
- IC1 pad 1: unconnected-(IC1-DPA2-Pad1) -> Net-(IC1-DPA2)
- IC1 pad 10: unconnected-(IC1-VBUSA1-Pad10) -> /PD_Control/VBUSA1
- IC1 pad 11: unconnected-(IC1-VBUSB-Pad11) -> Net-(IC1-VBUSB)
- IC1 pad 12: unconnected-(IC1-VBUSC-Pad12) -> /PD_Control/VBUSC
- IC1 pad 13: unconnected-(IC1-VOUTC-Pad13) -> /PD_Control/VOUTA1
- IC1 pad 14: unconnected-(IC1-VOUTA2-Pad14) -> Net-(IC1-VOUTA2)
- IC1 pad 15: unconnected-(IC1-VBUSA2-Pad15) -> Net-(IC1-VBUSA2)
- IC1 pad 16: unconnected-(IC1-VBUSL-Pad16) -> Net-(IC1-VBUSL)
- IC1 pad 17: unconnected-(IC1-BAT-Pad17) -> +BATT
- IC1 pad 18: unconnected-(IC1-NTC-Pad18) -> Net-(IC1-NTC)
- IC1 pad 19: unconnected-(IC1-VCC-Pad19) -> /PD_Control/VCC
- IC1 pad 2: unconnected-(IC1-SW_1-Pad2) -> /PD_Control/SW
- IC1 pad 20: unconnected-(IC1-KEY/GSET/IDA1-Pad20) -> Net-(IC1-KEY/GSET/IDA1)
- IC1 pad 21: unconnected-(IC1-FLED/BSET/IDA2-Pad21) -> Net-(D1-K)
- IC1 pad 22: unconnected-(IC1-LED5/CSET-Pad22) -> Net-(IC1-LED5/CSET)
- IC1 pad 23: unconnected-(IC1-LED4/I2C-Pad23) -> Net-(D6-A)
- IC1 pad 24: unconnected-(IC1-LED3/IRQ-Pad24) -> Net-(D4-K)
- IC1 pad 25: unconnected-(IC1-LED2/SDA-Pad25) -> Net-(D2-K)
- IC1 pad 26: unconnected-(IC1-LED1/SCK-Pad26) -> /PD_Control/DLED1
- IC1 pad 27: unconnected-(IC1-VOUTSP-Pad27) -> /PD_Control/VOUTA1
- IC1 pad 28: unconnected-(IC1-VOUTSN-Pad28) -> /PD_Control/VOUTSN
- IC1 pad 29: unconnected-(IC1-VOUT_1-Pad29) -> /PD_Control/VOUTSN
- IC1 pad 3: unconnected-(IC1-SW_2-Pad3) -> /PD_Control/SW
- IC1 pad 30: unconnected-(IC1-VOUT_2-Pad30) -> /PD_Control/VOUTSN
- IC1 pad 31: unconnected-(IC1-VOUT_3-Pad31) -> /PD_Control/VOUTSN
- IC1 pad 32: unconnected-(IC1-VOUT_4-Pad32) -> /PD_Control/VOUTSN
- IC1 pad 33: unconnected-(IC1-VOUT_5-Pad33) -> /PD_Control/VOUTSN
- IC1 pad 36: unconnected-(IC1-GATEA1-Pad36) -> /PD_Control/GATEA1
- IC1 pad 38: unconnected-(IC1-GATEC-Pad38) -> /PD_Control/GATEC
- IC1 pad 39: unconnected-(IC1-CCL/WLED-Pad39) -> Net-(IC1-CCL/WLED)
- IC1 pad 4: unconnected-(IC1-SW_3-Pad4) -> /PD_Control/SW
- IC1 pad 40: unconnected-(IC1-CC2-Pad40) -> /PD_Control/CC2
- IC1 pad 41: unconnected-(IC1-CC1-Pad41) -> /PD_Control/CC1
- IC1 pad 42: unconnected-(IC1-DMC-Pad42) -> /PD_Control/DC-
- IC1 pad 43: unconnected-(IC1-DPC-Pad43) -> /PD_Control/DC+
- IC1 pad 44: unconnected-(IC1-DMB-Pad44) -> Net-(IC1-DMB)
- IC1 pad 45: unconnected-(IC1-DPB-Pad45) -> Net-(IC1-DPB)
- IC1 pad 46: unconnected-(IC1-DMA1-Pad46) -> /PD_Control/DA-
- IC1 pad 47: unconnected-(IC1-DPA1-Pad47) -> /PD_Control/DA+
- IC1 pad 48: unconnected-(IC1-DMA2-Pad48) -> Net-(IC1-DMA2)
- IC1 pad 49: unconnected-(IC1-EP-Pad49) -> GND
- IC1 pad 5: unconnected-(IC1-SW_4-Pad5) -> /PD_Control/SW
- IC1 pad 6: unconnected-(IC1-SW_5-Pad6) -> /PD_Control/SW
- IC1 pad 7: unconnected-(IC1-BST-Pad7) -> /PD_Control/BST
- IC1 pad 8: unconnected-(IC1-DATA-Pad8) -> Net-(IC1-DATA)
- IC1 pad 9: unconnected-(IC1-VOUTA1-Pad9) -> /PD_Control/VOUTA1
- J1 pad 1: unconnected-(J1-VCC-Pad1) -> /PD_Control/VBUSA1
- J1 pad 2: unconnected-(J1-D--Pad2) -> /PD_Control/D-
- J1 pad 3: unconnected-(J1-D+-Pad3) -> /PD_Control/D+
- J1 pad 4: unconnected-(J1-GND-Pad4) -> GND
- J1 pad 5: unconnected-(J1-MH1-Pad5) -> GND
- J1 pad 6: unconnected-(J1-MH2-Pad6) -> GND
- J2 pad A1: unconnected-(J2-GND1-PadA1) -> GND
- J2 pad A12: unconnected-(J2-GND2-PadA12) -> GND
- J2 pad A4: unconnected-(J2-VBUS1-PadA4) -> /PD_Control/VBUSC
- J2 pad A5: unconnected-(J2-CC1-PadA5) -> /PD_Control/CC1
- J2 pad A6: unconnected-(J2-DA+-PadA6) -> /PD_Control/D1+
- J2 pad A7: unconnected-(J2-DA--PadA7) -> /PD_Control/D1-
- J2 pad A9: unconnected-(J2-VBUS2-PadA9) -> /PD_Control/VBUSC
- J2 pad B1: unconnected-(J2-GND3-PadB1) -> GND
- J2 pad B12: unconnected-(J2-GND4-PadB12) -> GND
- J2 pad B4: unconnected-(J2-VBUS3-PadB4) -> /PD_Control/VBUSC
- J2 pad B5: unconnected-(J2-CC2-PadB5) -> /PD_Control/CC2
- J2 pad B6: unconnected-(J2-DB+-PadB6) -> /PD_Control/D1+
- J2 pad B7: unconnected-(J2-DB--PadB7) -> /PD_Control/D1-
- J2 pad B9: unconnected-(J2-VBUS4-PadB9) -> /PD_Control/VBUSC
- J2 pad SH1: unconnected-(J2-SHIELD1-PadSH1) -> GND
- J2 pad SH2: unconnected-(J2-SHIELD2-PadSH2) -> GND
- J2 pad SH3: unconnected-(J2-SHIELD3-PadSH3) -> GND
- J2 pad SH4: unconnected-(J2-SHIELD4-PadSH4) -> GND
- L1 pad 1: +VDC -> +BATT

Commit message: randome one
Parts:
- C4, C5: moved to B.Cu
- moved R6 135.4 mm to (255.2, 142.8)
- moved U3 124.3 mm to (250.1, 133.0)
- moved R9 122.7 mm to (241.9, 142.7)
- moved R8 118.3 mm to (238.3, 136.0)
- moved Q3 116.0 mm to (236.9, 124.9)
- moved Q4 116.0 mm to (241.4, 124.9)
- moved R7 116.0 mm to (237.7, 119.1)
- moved TP12 116.0 mm to (231.6, 125.7)
- moved TP13 116.0 mm to (231.6, 131.7)
- moved C12 111.3 mm to (243.8, 129.6)
- moved R3 105.5 mm to (193.5, 140.1)
- moved C10 105.5 mm to (213.2, 58.7), turned to -90 degrees
- moved C8 100.4 mm to (209.5, 58.7), turned to -90 degrees
- moved C9 97.4 mm to (205.8, 58.7), turned to -90 degrees
- moved R5 96.4 mm to (179.1, 142.9)
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Connections:
- U1 pad 5: unconnected-(U1-VBUS-Pad5) -> /PD_Control/VBUSC
- U2 pad 5: unconnected-(U2-VBUS-Pad5) -> /PD_Control/VBUSA1
Routing:
- net /PD_Control/VBUSC: track 0.00 -> 21.3 mm, vias 0 -> 1
- net /PD_Control/VBUSA1: track 0.00 -> 13.3 mm, vias 0 -> 1
- net /PD_Control/D1-: track 0.00 -> 8.30 mm
- net /PD_Control/D1+: track 0.00 -> 8.30 mm
- net /PD_Control/D-: track 0.00 -> 7.48 mm
- net /PD_Control/D+: track 0.00 -> 7.48 mm
Other:
- board size 9.3 x 6 mm -> 6 x 9.3 mm

Commit message: halfway through pd everything
Parts:
- removed TP7: DPB, TestPoint:TestPoint_Pad_D1.0mm
- removed TP8: DMB, TestPoint:TestPoint_Pad_D1.0mm
- C4, C5: moved to F.Cu
- U1, U2: moved to B.Cu
- moved C10 78.1 mm to (144.1, 95.2), turned to 0 degrees
- moved C8 76.7 mm to (144.1, 98.8), turned to 0 degrees
- moved C9 75.5 mm to (144.1, 102.2), turned to 0 degrees
- moved R1 67.3 mm to (142.3, 90.8), turned to -90 degrees
- moved C7 61.7 mm to (146.0, 90.8), turned to 90 degrees
- moved C6 55.9 mm to (144.1, 86.0), turned to 0 degrees
- moved L1 40.9 mm to (146.4, 129.7)
- moved C3 15.9 mm to (143.5, 116.8)
- moved Q1 12.1 mm to (129.9, 119.2), turned to -90 degrees
- moved Q2 10.7 mm to (133.9, 94.5), turned to -90 degrees
- moved TP4 9.59 mm to (78.8, 96.7)
- moved TP9 8.66 mm to (98.8, 99.9)
- moved TP5 7.31 mm to (79.9, 105.0)
- moved IC1 7.00 mm to (143.0, 110.0), turned to 90 degrees
- moved TP10 6.88 mm to (97.0, 105.7)
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Connections:
- IC1 pad 44: Net-(IC1-DMB) -> unconnected-(IC1-DMB-Pad44)
- IC1 pad 45: Net-(IC1-DPB) -> unconnected-(IC1-DPB-Pad45)
- U1 pad 1: /PD_Control/D1+ -> /PD_Control/D1-
- U1 pad 3: /PD_Control/D1- -> /PD_Control/D1+
- U1 pad 4: /PD_Control/DC- -> /PD_Control/DC+
- U1 pad 6: /PD_Control/DC+ -> /PD_Control/DC-
- U2 pad 1: /PD_Control/D- -> /PD_Control/D+
- U2 pad 3: /PD_Control/D+ -> /PD_Control/D-
- U2 pad 4: /PD_Control/DA+ -> /PD_Control/DA-
- U2 pad 6: /PD_Control/DA- -> /PD_Control/DA+
Routing:
- net /PD_Control/VOUTA1: track 0.00 -> 47.8 mm, vias 0 -> 18
- net /PD_Control/CC2: track 0.00 -> 30.2 mm
- net /PD_Control/CC1: track 0.00 -> 21.7 mm
- net /PD_Control/GATEC: track 0.00 -> 19.2 mm, vias 0 -> 4
- net /PD_Control/GATEA1: track 0.00 -> 19.0 mm, vias 0 -> 4
- net /PD_Control/DC-: track 0.00 -> 18.4 mm, vias 0 -> 1
- net /PD_Control/DA+: track 0.00 -> 18.0 mm, vias 0 -> 1
- net /PD_Control/DA-: track 0.00 -> 17.7 mm, vias 0 -> 1
- net /PD_Control/DC+: track 0.00 -> 17.0 mm, vias 0 -> 1
- net /PD_Control/VBUSC: track 21.3 -> 4.56 mm, vias 1 -> 14
- net /PD_Control/VBUSA1: track 13.3 -> 7.68 mm
- net /PD_Control/VOUTSN: track 0.00 -> 3.97 mm
- net GND: vias 0 -> 9
- added copper zone on F.Cu, net /PD_Control/GATEA1
- added copper zone on F.Cu, net /PD_Control/VBUSA1
- added copper zone on B.Cu, net /PD_Control/VBUSC
- added copper zone on F.Cu, net /PD_Control/VBUSC
- added copper zone on B.Cu, net /PD_Control/VOUTA1
- added copper zone on F.Cu, net /PD_Control/VOUTA1
- added copper zone on F.Cu, net /PD_Control/VOUTSN
Other:
- board size 6 x 9.3 mm -> 48.7 x 69.6 mm
- board text added: "DC+"
- board text added: "DC-"

Commit message: mostly done on pd layout
Parts:
- removed TP10: DATA, TestPoint:TestPoint_Pad_D1.0mm
- removed TP9: VBUSB, TestPoint:TestPoint_Pad_D1.0mm
- D1, D2, D3, D4, D5, D6, R4, S1: moved to B.Cu
- moved S1 128.0 mm to (211.3, 107.0), turned to 180 degrees
- moved D2 123.8 mm to (208.8, 92.1), turned to 180 degrees
- moved D4 120.3 mm to (206.6, 101.6), turned to 180 degrees
- moved D5 110.4 mm to (200.5, 107.8), turned to 180 degrees
- moved D1 107.6 mm to (198.8, 86.8), turned to 180 degrees
- moved D3 97.8 mm to (192.2, 101.8), turned to 180 degrees
- moved D6 87.2 mm to (184.4, 101.8), turned to 180 degrees
- moved R4 79.5 mm to (177.7, 109.0), turned to 180 degrees
- moved R3 49.7 mm to (154.5, 109.4)
- moved R5 42.9 mm to (154.5, 107.8)
- moved C11 34.5 mm to (154.5, 112.6)
- moved R2 32.5 mm to (154.5, 111.0)
- moved TP1 28.7 mm to (175.0, 80.8)
- moved L1 4.76 mm to (147.0, 125.0), turned to 180 degrees
- moved C3 0.87 mm to (143.8, 116.0), turned to 90 degrees
Connections:
- IC1 pad 11: Net-(IC1-VBUSB) -> unconnected-(IC1-VBUSB-Pad11)
- IC1 pad 8: Net-(IC1-DATA) -> unconnected-(IC1-DATA-Pad8)
Routing:
- net /PD_Control/VOUTA1: track 47.8 -> 91.9 mm, vias 18 -> 20
- net /PD_Control/VBUSC: track 4.56 -> 29.1 mm
- net /PD_Control/VBUSA1: track 7.68 -> 30.8 mm, vias 1 -> 3
- net /PD_Control/VOUTSN: track 3.97 -> 21.8 mm
- net /PD_Control/VCC: track 0.00 -> 12.9 mm
- net Net-(IC1-KEY/GSET/IDA1): track 0.00 -> 8.30 mm
- net Net-(IC1-LED5/CSET): track 0.00 -> 7.97 mm
- net Net-(D1-K): track 0.00 -> 7.80 mm
- net /PD_Control/SW: track 0.00 -> 4.64 mm
- net /PD_Control/BST: track 0.00 -> 2.45 mm
- added copper zone on F.Cu, net /PD_Control/SW

Commit message: pc done
Parts:
- removed TP11: CCL/WLED, TestPoint:TestPoint_Pad_D1.0mm
- removed TP2: VBUSL, TestPoint:TestPoint_Pad_D1.0mm
- removed TP3: VBUSS2, TestPoint:TestPoint_Pad_D1.0mm
- removed TP4: VOUTA2, TestPoint:TestPoint_Pad_D1.0mm
- removed TP5: DMA2, TestPoint:TestPoint_Pad_D1.0mm
- removed TP6: DPA2, TestPoint:TestPoint_Pad_D1.0mm
- added H1: MountingHole, MountingHole:MountingHole_2.2mm_M2, F.Cu at (120.5, 130.0)
- C12, Q3, Q4, R6, R7, R8, R9, TP1, TP12, U3: moved to B.Cu
- moved R6 113.5 mm to (149.7, 100.8), turned to 180 degrees
- moved R9 108.2 mm to (143.0, 99.0), turned to -90 degrees
- moved U3 105.4 mm to (151.7, 95.1)
- moved Q4 100.4 mm to (146.5, 92.0)
- moved R8 99.1 mm to (151.0, 89.0), turned to 90 degrees
- moved C12 95.7 mm to (156.0, 91.4), turned to 180 degrees
- moved Q3 94.9 mm to (146.5, 96.0), turned to 180 degrees
- moved TP12 93.7 mm to (146.5, 86.5), turned to 180 degrees
- moved D2 88.4 mm to (128.0, 128.0), turned to 90 degrees
- moved R7 85.3 mm to (155.4, 96.7), turned to -90 degrees
- moved TP13 81.6 mm to (150.0, 129.0)
- moved D4 73.6 mm to (138.0, 128.0), turned to 90 degrees
- moved D1 65.4 mm to (143.0, 121.0), turned to -90 degrees
- moved D3 64.8 mm to (133.0, 128.0), turned to -90 degrees
- moved S1 62.9 mm to (150.0, 121.0), turned to 90 degrees
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Connections:
- net Net-(Q4-S_1) renamed /BMS/B-
- D2 pad 1: Net-(D2-K) -> /PD_Control/DLED1
- D2 pad 2: /PD_Control/DLED1 -> Net-(D2-A)
- D3 pad 1: /PD_Control/DLED1 -> Net-(D2-A)
- D3 pad 2: Net-(D2-K) -> /PD_Control/DLED1
- D4 pad 1: Net-(D4-K) -> /PD_Control/DLED1
- D4 pad 2: /PD_Control/DLED1 -> Net-(D4-A)
- D5 pad 1: /PD_Control/DLED1 -> Net-(D4-A)
- D5 pad 2: Net-(D4-K) -> /PD_Control/DLED1
- IC1 pad 1: Net-(IC1-DPA2) -> unconnected-(IC1-DPA2-Pad1)
- IC1 pad 14: Net-(IC1-VOUTA2) -> unconnected-(IC1-VOUTA2-Pad14)
- IC1 pad 15: Net-(IC1-VBUSA2) -> unconnected-(IC1-VBUSA2-Pad15)
- IC1 pad 16: Net-(IC1-VBUSL) -> unconnected-(IC1-VBUSL-Pad16)
- IC1 pad 24: Net-(D4-K) -> Net-(D4-A)
- IC1 pad 25: Net-(D2-K) -> Net-(D2-A)
- IC1 pad 39: Net-(IC1-CCL/WLED) -> unconnected-(IC1-CCL/WLED-Pad39)
- IC1 pad 48: Net-(IC1-DMA2) -> unconnected-(IC1-DMA2-Pad48)
- Q3 pad 1: /BMS/GND -> GND
- Q3 pad 2: /BMS/GND -> GND
- Q3 pad 3: /BMS/GND -> GND
- Q3 pad 5: Net-(Q3-D_1) -> /BMS/PowerNodeBMS
- Q3 pad 6: Net-(Q3-D_2) -> /BMS/PowerNodeBMS
- Q3 pad 7: Net-(Q3-D_3) -> /BMS/PowerNodeBMS
- Q3 pad 8: Net-(Q3-D_4) -> /BMS/PowerNodeBMS
- Q3 pad 9: (no net) -> /BMS/PowerNodeBMS
- Q4 pad 5: Net-(Q3-D_4) -> /BMS/PowerNodeBMS
- Q4 pad 6: Net-(Q3-D_3) -> /BMS/PowerNodeBMS
- Q4 pad 7: Net-(Q3-D_2) -> /BMS/PowerNodeBMS
- Q4 pad 8: Net-(Q3-D_1) -> /BMS/PowerNodeBMS
- Q4 pad 9: (no net) -> /BMS/PowerNodeBMS
- R6 pad 1: /BMS/VDC -> +BATT
- R7 pad 2: /BMS/GND -> GND
- R9 pad 2: /BMS/GND -> GND
- TP13 pad 1: /BMS/VDC -> +BATT
Routing:
- net /PD_Control/DLED1: track 0.00 -> 55.7 mm, vias 0 -> 1
- net +BATT: track 0.00 -> 47.5 mm
- net Net-(D2-A): track 0.00 -> 38.7 mm, vias 0 -> 1
- net Net-(D4-A): track 0.00 -> 35.9 mm, vias 0 -> 1
- net Net-(D6-A): track 0.00 -> 30.1 mm, vias 0 -> 1
- net Net-(D1-K): track 7.80 -> 18.1 mm, vias 0 -> 1
- net Net-(IC1-NTC): track 0.00 -> 7.31 mm
- net /PD_Control/VCC: track 12.9 -> 19.9 mm, vias 0 -> 1
- net Net-(IC1-KEY/GSET/IDA1): track 8.30 -> 14.5 mm, vias 0 -> 1
- net GND: track 0.00 -> 3.58 mm, vias 9 -> 10
- net Net-(IC1-LED5/CSET): track 7.97 -> 4.97 mm
- net /PD_Control/VOUTA1: track 91.9 -> 93.5 mm
- net /PD_Control/VOUTSN: track 21.8 -> 23.2 mm
- net /PD_Control/VBUSA1: track 30.8 -> 32.1 mm
- net /PD_Control/GATEA1: track 19.0 -> 19.6 mm
- added copper zone on F.Cu, net +BATT
- added copper zone on B.Cu, net Net-(Q4-G)
Other:
- board size 48.7 x 69.6 mm -> 44 x 53 mm

Commit message: added logo
Routing:
- added copper zone on B.Cu, net GND
- added copper zone on F.Cu, net GND
- added copper zone on B.Cu, net Net-(Q3-G)
Changed lines of the file:
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@@
+	)
+	(segment
+		(start 129.2847 113.5)
+		(end 129.2847 113.4885)
+		(width 0.6)
+		(layer "F.Cu")
+		(net 20)
 	)
 	(segment
@@
 	)
 	(segment
-		(start 129.2847 113.5)
-		(end 134.5847 108.2)
+		(start 129.2847 113.4885)
+		(end 134.5732 108.2)
+		(width 0.6)
+		(layer "F.Cu")
+		(net 20)
+	)
+	(segment
+		(start 134.5732 108.2)
+		(end 139.1412 108.2)
 		(width 0.6)
 		(layer "F.Cu")
@@
 		(end 129.2847 116.5)
 		(width 0.5)
-		(layer "F.Cu")
-		(net 20)
-	)
-	(segment
-		(start 134.5847 108.2)
-		(end 139.1412 108.2)
-		(width 0.6)
 		(layer "F.Cu")
 		(net 20)
@@
 		(name "1")
 		(hatch edge 0.5)
+		(priority 1)
 		(connect_pads yes
 			(clearance 0)
@@
 		(polygon
 			(pts
-				(xy 123.6218 120.101354) (xy 123.952 120.0912) (xy 125.1712 118.872) (xy 129.4638 118.872) (xy 129.489464 123.7996)
-				(xy 123.6218 123.7996)
+				(xy 123.6218 120.101354) (xy 123.820971 120.095229) (xy 125.0442 118.872) (xy 129.4638 118.872)
+				(xy 129.489464 123.7996) (xy 123.6218 123.7996)
 			)
 		)
@@
 		(min_thickness 0.25)
 		(filled_areas_thickness no)
-		(fill
+		(fill yes
 			(thermal_gap 0.5)
 			(thermal_bridge_width 0.5)
@@
 		(name "1")
 		(hatch edge 0.5)
+		(priority 1)
 		(connect_pads yes
 			(clearance 0)
@@
 			(pts
 				(xy 141.9098 107.5436) (xy 141.9098 106.5022) (xy 141.52873 106.218067) (xy 141.52873 91.679346)
-				(xy 143.890941 91.679346) (xy 143.891002 104.0638) (xy 143.7132 106.5276) (xy 143.7132 107.5436)
+				(xy 143.890941 91.679346) (xy 143.891002 103.9876) (xy 143.7132 104.1908) (xy 143.7132 106.5276)
+				(xy 143.7132 107.5436)
 			)
 		)
@@
 	)
 	(zone
+		(net 2)
+		(net_name "GND")
+		(layer "F.Cu")
+		(name "24")
+		(hatch edge 0.5)
+		(connect_pads yes
+			(clearance 0)
+		)
+		(min_thickness 0.25)
+		(filled_areas_thickness no)
+		(fill yes
+			(thermal_gap 0.5)
+			(thermal_bridge_width 0.5)
+			(island_removal_mode 2)
+			(island_area_min 10)
+		)
+		(polygon
+			(pts
+				(xy 114.9858 104.5464) (xy 159.004 104.5718) (xy 159.004 125.7808) (xy 137.4394 125.7808) (xy 137.4394 134.0104)
+				(xy 115.0112 134.0104)
+			)
+		)
+	)
+	(zone
 		(net 22)
 		(net_name "/PD_Control/GATEA1")
@@
 		(polygon
 			(pts
-				(xy 128.1684 111.3028) (xy 129.117893 112.211299) (xy 133.13505 108.3564) (xy 133.1214 106.3752)
+				(xy 128.1684 111.3028) (xy 128.930717 112.032205) (xy 133.132595 108.000046) (xy 133.1214 106.3752)
 				(xy 132.3086 105.0798) (xy 127.21685 110.049492)
 			)
@@
 	)
 	(zone
+		(net 2)
+		(net_name "GND")
+		(layer "B.Cu")
+		(name "1")
+		(hatch edge 0.5)
+		(connect_pads yes
+			(clearance 0)
+		)
+		(min_thickness 0.25)
+		(filled_areas_thickness no)
+		(fill yes
+			(thermal_gap 0.5)
+			(thermal_bridge_width 0.5)
+			(island_removal_mode 2)
+			(island_area_min 10)
+		)
+		(polygon
+			(pts
+				(xy 159.004 104.5718) (xy 159.004 134.0104) (xy 114.9858 134.0104) (xy 114.9858 104.5464)
+			)
+		)
+	)
+	(zone
+		(net 42)
+		(net_name "Net-(Q3-G)")
+		(layer "B.Cu")
+		(name "45")
+		(hatch edge 0.5)
+		(connect_pads yes
+			(clearance 0)
+		)
+		(min_thickness 0.25)
+		(filled_areas_thickness no)
+		(fill yes
+			(thermal_gap 0.5)
+			(thermal_bridge_width 0.5)
+		)
+		(polygon
+			(pts
+				(xy 145.706784 96.929083) (xy 145.706784 97.894283) (xy 143.6784 98.298) (xy 141.9258 98.298) (xy 141.922184 96.598883)
+				(xy 143.6784 96.5962)
+			)
+		)
+	)
+	(zone
+		(net 5)
+		(net_name "/PD_Control/VBUSC")
+		(layer "B.Cu")
+		(name "1")
+		(hatch edge 0.5)
+		(priority 2)
+		(connect_pads yes
+			(clearance 0)
+		)
+		(min_thickness 0.025)
+		(filled_areas_thickness no)
+		(fill yes
+			(thermal_gap 0.5)
+			(thermal_bridge_width 0.5)
+		)
+		(polygon
+			(pts
+				(xy 121.031 119.1514) (xy 121.031 118.5926) (xy 123.19 118.5926) (xy 127.762 118.5926) (xy 127.762 119.5832)
+				(xy 126.7206 120.3198) (xy 123.987338 120.3198) (xy 122.971338 119.1514)
+			)
+		)
+	)
+	(zone
 		(net 43)
 		(net_name "Net-(Q4-G)")
@@
 		(min_thickness 0.25)
 		(filled_areas_thickness no)
-		(fill
-			(thermal_gap 0.5)
-			(thermal_bridge_width 0.5)
-		)
-		(polygon
-			(pts
-				(xy 145.706784 96.929083) (xy 145.706784 97.894283) (xy 143.6784 98.298) (xy 141.9258 98.298) (xy 141.922184 96.598883)
-				(xy 143.6784 96.5962)
-			)
-		)
-	)
-	(zone
-		(net 5)
-		(net_name "/PD_Control/VBUSC")
-		(layer "B.Cu")
-		(name "1")
-		(hatch edge 0.5)
-		(priority 2)
-		(connect_pads yes
-			(clearance 0)
-		)
-		(min_thickness 0.025)
-		(filled_areas_thickness no)
-		(fill yes
-			(thermal_gap 0.5)
-			(thermal_bridge_width 0.5)
-		)
-		(polygon
-			(pts
-				(xy 121.031 119.1514) (xy 121.031 118.5926) (xy 123.19 118.5926) (xy 127.762 118.5926) (xy 127.762 119.5832)
-				(xy 126.7206 120.3198) (xy 123.987338 120.3198) (xy 122.971338 119.1514)
-			)
-		)
-	)
-	(zone
-		(net 43)
-		(net_name "Net-(Q4-G)")
-		(layer "B.Cu")
-		(hatch edge 0.5)
-		(priority 12)
-		(connect_pads yes
-			(clearance 0)
-		)
-		(min_thickness 0.25)
-		(filled_areas_thickness no)
-		(fill
-			(thermal_gap 0.5)
-			(thermal_bridge_width 0.5)
+		(fill yes
+			(thermal_gap 0.5)
+			(thermal_bridge_width 0.5)

Commit message: mostly ddone
Parts:
- Q4, R8, TP12: moved to F.Cu
- moved R6 11.4 mm to (155.5, 91.0), turned to 90 degrees
- moved Q4 9.01 mm to (155.0, 95.0), turned to 180 degrees
- moved TP12 7.65 mm to (154.0, 88.0)
- moved C12 7.64 mm to (149.0, 88.5)
- moved R7 7.37 mm to (152.2, 90.0), turned to 90 degrees
- moved Q3 5.09 mm to (150.0, 99.7), turned to 90 degrees
- moved R9 4.72 mm to (147.0, 96.5), turned to 180 degrees
- moved U3 3.99 mm to (150.0, 91.5), turned to 90 degrees
- moved R8 3.54 mm to (151.5, 92.5)
Routing:
- net +BATT: track 47.5 -> 59.8 mm, vias 0 -> 2
- net /BMS/B-: track 0.00 -> 8.27 mm, vias 0 -> 2
- net Net-(U3-BAT): track 0.00 -> 6.12 mm
- net Net-(Q3-G): track 0.00 -> 5.03 mm
- net Net-(Q4-G): track 0.00 -> 2.51 mm, vias 0 -> 2
- net Net-(U3-V-): track 0.00 -> 1.75 mm
- net GND: vias 10 -> 143
- net /BMS/PowerNodeBMS: vias 0 -> 18
- added copper zone on F.Cu, net /BMS/B-
- added copper zone on B.Cu, net /BMS/PowerNodeBMS
- added copper zone on F.Cu, net /BMS/PowerNodeBMS
- added copper zone on F.Cu, net Net-(Q4-G)
- removed copper zone on B.Cu, net Net-(Q4-G)

Commit message: mostly done
Parts:
- added G***: LOGO, LOGO, B.Cu at (146.3, 105.9)
- added G***: LOGO, LOGO, B.Cu at (133.6, 85.9)
- U3: value BQ297xy -> BQ29700
- moved C3 0.70 mm to (143.2, 115.6)
- moved R8 0.20 mm to (151.3, 92.5)
Routing:
- net Net-(D1-A): track 0.37 -> 3.13 mm
- net Net-(U3-BAT): track 6.12 -> 8.55 mm
- net /PD_Control/BST: track 2.45 -> 1.76 mm
- net /PD_Control/SW: track 4.64 -> 3.98 mm
Other:
- board text added: "Arafat Babar"
- board text added: "Designed by :"
- board text added: "Designed for 1S3p with 21700 0.48Ah each"
- board text added: "LI-ION BATTERY RISK OF FIRE OR EXPLOSION DO NOT SHORT, CRUSH, OR OVERCHARGE"
- board text added: "Portable Power Bank"
- board text added: "SW6208"
- board text added: "Turning schematics into copper."
- board text added: "Warning Risk of Fire Handle Carefully"
