File: PortablePower/PortablePower.kicad_pcb (KiCad board)
At the start: 2 copper layers, 44 x 53 mm, 45 parts, among them IC1 SW6208, J1 USB1130-15-A, J2 2137160001, Q1 CSD17313Q2, Q2 CSD17313Q2, Q3 CSD16406Q3, Q4 CSD16406Q3, U1 USBLC6-2SC6, U2 USBLC6-2SC6, U3 BQ29700

Commit message: final update
Parts:
- C12, C7: footprint Capacitor_SMD:C_0805_2012Metric_Pad1.18x1.45mm_HandSolder -> Capacitor_SMD:C_0603_1608Metric_Pad1.08x0.95mm_HandSolder
- R1: footprint Resistor_SMD:R_1206_3216Metric_Pad1.30x1.75mm_HandSolder -> Resistor_SMD:R_2512_6332Metric_Pad1.40x3.35mm_HandSolder
- U3: value BQ29700 -> BQ297xy
- moved C7 4.11 mm to (141.9, 88.7)
- moved R1 3.52 mm to (145.5, 87.4)
- moved C12 0.17 mm to (149.1, 88.4)
Routing:
- net /PD_Control/VOUTSN: track 23.2 -> 19.6 mm
- net GND: vias 143 -> 140
