File: PortablePower/BMS.kicad_sch (KiCad schematic)
At the start: 0 parts

Commit message: schematic complete
Parts:
- added C12: 0.1uf, symbol Device:C
- added Q3, Q4: CSD16406Q3, DQG_VSON-CLIP, symbol CSD16406Q3:CSD16406Q3
- added R6: 330, Resistor_SMD:R_0805_2012Metric_Pad1.20x1.40mm_HandSolder, symbol Device:R
- added R7: 2.2k, symbol Device:R
- added R8, R9: 5M, Resistor_SMD:R_1206_3216Metric_Pad1.30x1.75mm_HandSolder, symbol Device:R
- added TP12: B-, TestPoint:TestPoint_Pad_D4.0mm, symbol Connector:TestPoint
- added TP13: B+, TestPoint:TestPoint_Pad_4.0x4.0mm, symbol Connector:TestPoint
- added U3: BQ297xy, Package_SON:WSON-6_1.5x1.5mm_P0.5mm, symbol Battery_Management:BQ297xy
Connections:
- new net: Q4.4 (G), R8.1, U3.3 (Dout)
- new net: C12.2, Q4.1 (S_1), Q4.2 (S_2), Q4.3 (S_3), R8.2, TP12.1, U3.4 (VSS)
- new net: R7.1, U3.6 (V-)
- new net: C12.1, R6.2, U3.5 (BAT)
- new net: Q3.4 (G), R9.1, U3.2 (Cout)
- new net: Q3.8 (D_4), Q4.5 (D_1)
- new net: Q3.7 (D_3), Q4.6 (D_2)
- new net: Q3.6 (D_2), Q4.7 (D_3)
- new net: Q3.5 (D_1), Q4.8 (D_4)
- new net GND: Q3.1 (S_1), Q3.2 (S_2), Q3.3 (S_3), R7.2, R9.2
- new net VDC: R6.1, TP13.1

Commit message: before done schematic
Parts:
- C12: footprint (none) -> Capacitor_SMD:C_0805_2012Metric_Pad1.18x1.45mm_HandSolder
- R7: footprint (none) -> Resistor_SMD:R_0603_1608Metric_Pad0.98x0.95mm_HandSolder
Changed lines of the file:
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@@
 			)
 		)
-		(property "Footprint" ""
+		(property "Footprint" "Resistor_SMD:R_0603_1608Metric_Pad0.98x0.95mm_HandSolder"
 			(at 53.467 61.595 90)
 			(effects
@@
 			)
 		)
-		(property "Footprint" ""
+		(property "Footprint" "Capacitor_SMD:C_0805_2012Metric_Pad1.18x1.45mm_HandSolder"
 			(at 150.8252 64.135 0)
 			(effects

Commit message: randome one
Parts:
- R8, R9: now not fitted
Changed lines of the file:
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@@
 		(in_bom yes)
 		(on_board yes)
-		(dnp no)
+		(dnp yes)
 		(fields_autoplaced yes)
 		(property "Reference" "R8"
@@
 		(in_bom yes)
 		(on_board yes)
-		(dnp no)
+		(dnp yes)
 		(fields_autoplaced yes)
 		(property "Reference" "R9"

Commit message: pc done
Parts:
- Q3, Q4: footprint DQG_VSON-CLIP -> CSD16406Q3:DQG_VSON-CLIP
Connections:
- net B-: now reaches C12.2, Q4.1 (S_1), Q4.2 (S_2), Q4.3 (S_3), R8.2, TP12.1, U3.4 (VSS)
- net PowerNodeBMS: now reaches Q3.8 (D_4), Q4.5 (D_1)
- net PowerNodeBMS: now also Q3.5 (D_1), Q3.6 (D_2), Q3.7 (D_3), Q4.6 (D_2), Q4.7 (D_3), Q4.8 (D_4)
Changed lines of the file:
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@@
 	(paper "A5")
 	(junction
+		(at 89.535 79.375)
+		(diameter 0)
+		(color 0 0 0 0)
+	)
+	(junction
 		(at 120.015 80.645)
 		(diameter 0)
@@
 	)
 	(junction
+		(at 89.535 81.915)
+		(diameter 0)
+		(color 0 0 0 0)
+	)
+	(junction
 		(at 149.86 53.975)
 		(diameter 0)
@@
 	)
 	(junction
+		(at 89.535 76.835)
+		(diameter 0)
+		(color 0 0 0 0)
+	)
+	(junction
 		(at 55.245 78.105)
 		(diameter 0)
@@
 	)
 	(junction
+		(at 89.535 84.455)
+		(diameter 0)
+		(color 0 0 0 0)
+	)
+	(junction
 		(at 75.565 69.215)
 		(diameter 0)
@@
 	(wire
 		(pts
+			(xy 89.535 81.915) (xy 89.535 84.455)
+		)
+		(stroke
+			(width 0)
+			(type default)
+		)
+	)
+	(wire
+		(pts
 			(xy 103.505 60.325) (xy 120.65 60.325)
 		)
@@
 	(wire
 		(pts
+			(xy 89.535 79.375) (xy 89.535 81.915)
+		)
+		(stroke
+			(width 0)
+			(type default)
+		)
+	)
+	(wire
+		(pts
+			(xy 89.535 76.835) (xy 89.535 79.375)
+		)
+		(stroke
+			(width 0)
+			(type default)
+		)
+	)
+	(wire
+		(pts
 			(xy 149.86 43.815) (xy 149.86 38.1)
 		)
@@
 		)
 	)
+	(label "B-"
+		(at 143.51 78.105 0)
+		(effects
+			(font
+				(size 1.27 1.27)
+			)
+			(justify left bottom)
+		)
+	)
+	(label "PowerNodeBMS"
+		(at 89.535 76.835 90)
+		(effects
+			(font
+				(size 1.27 1.27)
+			)
+			(justify left bottom)
+		)
+	)
 	(hierarchical_label "VDC"
-		(shape input)
+		(shape output)
 		(at 49.53 38.1 180)
 		(effects
@@
 	)
 	(hierarchical_label "GND"
-		(shape input)
+		(shape output)
 		(at 49.53 78.105 180)
 		(effects
@@
 			)
 		)
-		(property "Footprint" "DQG_VSON-CLIP"
+		(property "Footprint" "CSD16406Q3:DQG_VSON-CLIP"
 			(at 111.125 171.755 0)
 			(effects
@@
 			)
 		)
-		(property "Footprint" "DQG_VSON-CLIP"
+		(property "Footprint" "CSD16406Q3:DQG_VSON-CLIP"
 			(at 83.185 171.755 0)
 			(effects

Commit message: mostly ddone
Other:
- company: (none) -> Mekatra
- title: (none) -> Battery Protection
Changed lines of the file:
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@@
 	(generator_version "9.0")
 	(paper "A5")
+	(title_block
+		(title "Battery Protection")
+		(date "2026-01-13")
+		(rev "1")
+		(company "Mekatra")
+		(comment 1 "BQ29700DSER")
+		(comment 2 "CSD16406Q3")
+	)
 	(junction
 		(at 89.535 79.375)
@@
 					(unit 1)
 				)
+			)
+		)
+	)
+	(symbol
+		(lib_id "Mekatra symbol kicad:LOGO")
+		(at 50.8 118.11 0)
+		(unit 1)
+		(exclude_from_sim no)
+		(in_bom yes)
+		(on_board yes)
+		(dnp no)
+		(fields_autoplaced yes)
+		(property "Reference" "#G2"
+			(at 50.8 111.1576 0)
+			(effects
+				(font
+					(size 1.27 1.27)
+				)
+				(hide yes)
+			)
+		)
+		(property "Value" "LOGO"
+			(at 50.8 125.0624 0)
+			(effects
+				(font
+					(size 1.27 1.27)
+				)
+				(hide yes)
+			)
+		)
+		(property "Footprint" ""
+			(at 50.8 118.11 0)
+			(effects
+				(font
+					(size 1.27 1.27)
+				)
+				(hide yes)
+			)
+		)
+		(property "Datasheet" ""
+			(at 50.8 118.11 0)
+			(effects
+				(font
+					(size 1.27 1.27)
+				)
+				(hide yes)
+			)
+		)
+		(property "Description" ""
+			(at 50.8 118.11 0)
+			(effects
+				(font
+					(size 1.27 1.27)
+				)
+				(hide yes)
+			)
+		)
+		(instances
+			(project "PortablePower"
+				(path "/4474177b-2e5c-4472-8e6c-d549a0d6c1d6/96561ace-f42a-4833-93f0-b23748914e58"
+					(reference "#G2")
+					(unit 1)
+				)

Commit message: final update
Parts:
- C12: footprint Capacitor_SMD:C_0805_2012Metric_Pad1.18x1.45mm_HandSolder -> Capacitor_SMD:C_0603_1608Metric_Pad1.08x0.95mm_HandSolder
Changed lines of the file:
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@@
 			)
 		)
-		(property "Footprint" "Capacitor_SMD:C_0805_2012Metric_Pad1.18x1.45mm_HandSolder"
+		(property "Footprint" "Capacitor_SMD:C_0603_1608Metric_Pad1.08x0.95mm_HandSolder"
 			(at 150.8252 64.135 0)
 			(effects
