File: PortablePower/pdcontrol.kicad_sch (KiCad schematic)
At the start: 33 parts, among them IC1 SW6208, J1 USB1130-15-A, J2 2137160001, Q1 CSD17313Q2, Q2 CSD17313Q2, U1 USBLC6-2SC6, U2 USBLC6-2SC6

Commit message: mostly done
Parts:
- IC1: footprint QFN40P600X600X80-49N -> SW6208:QFN40P600X600X80-49N
Changed lines of the file:
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@@
 			)
 		)
-		(property "Footprint" "QFN40P600X600X80-49N"
+		(property "Footprint" "SW6208:QFN40P600X600X80-49N"
 			(at 163.195 136.83 0)
 			(effects

Commit message: final update
Parts:
- C7: footprint Capacitor_SMD:C_0805_2012Metric_Pad1.18x1.45mm_HandSolder -> Capacitor_SMD:C_0603_1608Metric_Pad1.08x0.95mm_HandSolder
- R1: footprint Resistor_SMD:R_1206_3216Metric_Pad1.30x1.75mm_HandSolder -> Resistor_SMD:R_2512_6332Metric_Pad1.40x3.35mm_HandSolder
Changed lines of the file:
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@@
 			)
 		)
-		(property "Footprint" "Capacitor_SMD:C_0805_2012Metric_Pad1.18x1.45mm_HandSolder"
+		(property "Footprint" "Capacitor_SMD:C_0603_1608Metric_Pad1.08x0.95mm_HandSolder"
 			(at 119.38 164.7952 0)
 			(effects
@@
 			)
 		)
-		(property "Footprint" "Resistor_SMD:R_1206_3216Metric_Pad1.30x1.75mm_HandSolder"
+		(property "Footprint" "Resistor_SMD:R_2512_6332Metric_Pad1.40x3.35mm_HandSolder"
 			(at 123.19 177.038 90)
 			(effects
